Commit message: Working on the robot description

File: robot_description/robots/robco19e_with_Mover4.urdf.xacro (robot description, xacro)
@@ -16,5 +16,5 @@
   <xacro:include filename="$(find robot_description)/urdf/robco_imu_macro.xacro" />
   <xacro:include filename="$(find robot_description)/urdf/robco_rplidar_macro.xacro" />
-  <!--<xacro:include filename="$(find robot_description)/urdf/robco_mover4_macro.xacro" />-->
+  <xacro:include filename="$(find robot_description)/urdf/robco_mover4_macro.xacro" />
   <xacro:include filename="$(find robot_description)/urdf/robco_kinect_mount_macro.xacro" />
 <!--###################################################################################-->
@@ -28,9 +28,13 @@
 <xacro:robco_imu/>
 <!--Visual for the IMU mount point comment out !!!!!!!!!!!!!!!!!!!!!!!!!!!!!!!!!!!!!!!!!!!!!!!!!!!!!!!!!!!!!!!!-->
-  <xacro:robco_mountpoint_visualizer_box parent="base_link" device_name="imu" lenght= "${0.01}" width="${0.01}" height="${0.01}" x_loc="${0.0}" y_loc="${0.0}" z_loc="${round_plate_height}"/>
+  <xacro:robco_mountpoint_visualizer_box parent="base_link" device_name="imu" lenght= "${0.01}" width="${0.01}" height="${0.01}" x_loc="${0.0}" y_loc="${0.0}" z_loc="${0.04}"/>
 <!--########### ADD RPLIDAR A2  #############################-->
 <xacro:robco_rplidar_a2/>
 <!--Visual for the RPLidar A2 mount point comment out !!!!!!!!!!!!!!!!!!!!!!!!!!!!!!!!!!!!!!!!!!!!!!!!!!!!!!!!!!!!!!!!-->
   <xacro:robco_mountpoint_visualizer_box parent="second_deck" device_name="laser" lenght= "${0.01}" width="${0.01}" height="${0.01}" x_loc="${rplidar_X_offset}" y_loc="${rplidar_Y_offset}" z_loc="${rplidar_Z_offset}"/>
+<!--########### ADD MOVER 4 ARM  #############################-->
+<xacro:robco_mover4/>
+<!--Visual for the mover4 mount point comment out !!!!!!!!!!!!!!!!!!!!!!!!!!!!!!!!!!!!!!!!!!!!!!!!!!!!!!!!!!!!!!!!-->
+  <xacro:robco_mountpoint_visualizer_box parent="third_deck" device_name="mover4_arm" lenght= "${round_plate_height}" width="${round_plate_height}" height="${round_plate_height}" x_loc="${mover4_X_offset}" y_loc="${mover4_Y_offset}" z_loc="${mover4_Z_offset}"/>
 <!--########### ADD KINECT  #############################-->
 <xacro:robco_kinect />

File: robot_description/urdf/robco_2wd_base_macro.xacro (robot description, xacro)
@@ -34,5 +34,5 @@
         <turnGravityOff>false</turnGravityOff>
     </gazebo>
-  <!-- JOINT BASE_LINK TO BASE_FRAME-->
+  <!-- JOINT BASE_LINK TO BASE_FOOTPRINT-->
   <joint name="base_footprint_base_link_joint" type="fixed">
     <origin rpy="0 0 0" xyz="0 0 ${base_plate_botom_from_base_frame_Z_offset}"/>

File: robot_description/urdf/robco_imu_macro.xacro (robot description, xacro)
@@ -4,7 +4,12 @@
 <!-- Created by Stefan -->
 <!-- Service Robotics Group - Bulgaria - Version 1.0 from Oct. 11th, 2018. -->
+<!--Modified on 29.3.2019 - Mount the IMU based on base_link coordinates -->
 <xacro:include filename="$(find robot_description)/urdf/sensors/imu_macro.xacro" />
+<!--imu_link is used in the navigation stack - it should represent the center of the IMU chip-->
+<!--This mount point sets the imu_link position on the robot-->
 <xacro:macro name="robco_imu">
-<xacro:imu parent="third_deck" x_loc="${0}" y_loc="${0}" z_loc="${0}"/>
+<!--<xacro:imu parent="third_deck" x_loc="${0}" y_loc="${0}" z_loc="${0}"/>-->
+<!--For now the IMU is mounted in the center, on top of the base plate, which is round_plate_height over the base_link point-->
+<xacro:imu parent="base_link" x_loc="${0}" y_loc="${0}" z_loc="${round_plate_height}"/>
 </xacro:macro>
 </robot>

File: robot_description/urdf/robco_properties.xacro (robot description, xacro)
@@ -10,5 +10,6 @@
   <!--<xacro:property name="M_PI" value="3.1415926535897931" />-->
   <xacro:property name="M_PI_2" value="1.570796327" />
-  <xacro:property name="ROTATE_90_DEGREES" value="1.570796327" />
+  <xacro:property name="ROTATE_90_DEGREES" value="${M_PI_2}" />
+  <xacro:property name="ROTATE_180_DEGREES" value="${M_PI}" />
   <xacro:property name="DEG_TO_RAD" value="0.017453293" />
   <xacro:property name="SCALE_in_to_m" value="0.0254"/> <!--inches to meters-->

File: robot_description/urdf/sensors/imu_macro.xacro (robot description, xacro)
@@ -5,4 +5,5 @@
 <!-- Service Robotics Group - Bulgaria -  Version 1.0 from Oct. 9th, 2018. -->
   <xacro:macro name="imu" params="parent x_loc y_loc z_loc">
+<!--imu_link is used in the navigation stack - it should represent the center of the IMU chip-->
   <joint name="imu_joint" type="fixed">
     <origin xyz="${x_loc} ${y_loc} ${z_loc}" rpy="0 0 0" />

File: robot_description/urdf/sensors/rplidar_a2_macro.xacro (robot description, xacro)
@@ -6,7 +6,13 @@
 <xacro:macro name="rplidar_a2" params="parent x_loc y_loc z_loc mesh_offset_X mesh_offset_Y mesh_offset_Z">
     <joint name="rplidar_a2_joint" type="fixed">
-      <origin xyz="${x_loc} ${y_loc} ${z_loc}" rpy="0 0 0" />
+      <!--<origin xyz="${x_loc} ${y_loc} ${z_loc}" rpy="0 0 0" />-->
+      <!--Working parameters set for the static_transform_publisher -->
+      <!--<node pkg="tf2_ros" type="static_transform_publisher" name="base_link_to_laser" args="0.1876 0 0.178 0 3.14159 3.14159   /base_link /laser"/>-->
+      <origin xyz="${x_loc} ${y_loc} ${z_loc}" rpy="0 ${ROTATE_180_DEGREES} ${ROTATE_180_DEGREES}" />
       <parent link="${parent}"/>
-      <child link="rplidar_laser_beam_plane" />
+      <!--This link represents the laser beam plane and orientation-->
+      <!--Cahnge the name to laser as this name is used in the navigation stack-->
+      <!--<child link="rplidar_laser_beam_plane" />-->
+      <child link="laser" />
     </joint>
   <!--<joint name="rplidar_joint" type="fixed">
@@ -16,5 +22,6 @@
   </joint>-->
   <!-- rplidar Laser -->
-  <link name="rplidar_laser_beam_plane">
+  <!--<link name="rplidar_laser_beam_plane">-->
+  <link name="laser">
       <collision>
       <origin xyz="0 0 0" rpy="0 0 0"/>
@@ -26,4 +33,5 @@
     <visual>
     <!--Looks like the rplidar mesh is not with the correct diameter, modifying the Y offset in order to show the visual "almost" correctly -->
+      <!--<origin xyz="${mesh_offset_X} ${mesh_offset_Y} ${mesh_offset_Z}" rpy="0 0 0" />-->
       <origin xyz="${mesh_offset_X} ${mesh_offset_Y} ${mesh_offset_Z}" rpy="0 0 0" />
       <geometry>
